File: pcb/nrf-beacon.brd (EAGLE design)
At the start: 45 x 35 mm, 63 parts, among them CON1 NRF24-MODULE, CON3 MICRO-USB, IC1 STM32F303CCT6, IC2 LD39080, IC5 STC4054, Q2 25MHz, U1 SN65HVD230, X1 SWDABGEWINKELT, X2 SERIAL_DEBUG_3PINL

Commit message: pcb: add forgotten signal for monitoring charger
Connections:
- net CHARGER_CHRG: now also IC1.42
- net CHARGER_PROG: now also IC1.10
Routing:
- net CHARGER_PROG: track 1.26 -> 37.6 mm, vias 0 -> 2
- net CHARGER_CHRG: track 6.65 -> 31.0 mm, vias 0 -> 2
- net GND: track 260.1 -> 257.6 mm
- net N$2: track 38.0 -> 39.7 mm
- net DEBUG_RX: track 18.7 -> 19.6 mm
- net DEBUG_TX: track 20.2 -> 21.1 mm
- net VCC: track 29.4 -> 30.0 mm
- net SWDIO: track 28.0 -> 27.5 mm
