File: pcb/nrf-beacon.sch (EAGLE design)
At the start: 63 parts, among them CON1 NRF24-MODULE, CON3 MICRO-USB, IC1 STM32F303CCT6, IC2 LD39080, IC5 STC4054, Q2 25MHz, U1 SN65HVD230, X1 SWDABGEWINKELT, X2 SERIAL_DEBUG_3PINL

Commit message: pcb: add forgotten signal for monitoring charger
Connections:
- net CHARGER_CHRG: now also IC1PORTB_L.PB6
- net CHARGER_PROG: now also IC1PORTA_L.PA0
Other:
- note removed: "Errata: Forgot to connect CHARGER_CHRG and CHARGER_PROG to STM32 STC4054 seems to enter trickle-charge mode when connected to USB while battery is disconnected, so maybe connect V_BAT and VCC each over a diode to LDO to avoid low voltage operation"
- moved on the sheet: IC1PORTA_L
Changed lines of the file:
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@@
 <wire x1="162.56" y1="66.04" x2="193.04" y2="66.04" width="0.1524" layer="97"/>
 <wire x1="71.12" y1="109.22" x2="71.12" y2="127" width="0.1524" layer="97"/>
-<text x="17.78" y="185.42" size="1.778" layer="97">Errata:
-Forgot to connect CHARGER_CHRG
-and CHARGER_PROG to STM32
-STC4054 seems to enter trickle-charge
-mode when connected to USB while
-battery is disconnected, so maybe
-connect V_BAT and VCC each over a
-diode to LDO to avoid low voltage
-operation</text>
 </plain>
 <instances>
 <instance part="FRAME1" gate="G$1" x="0" y="0"/>
-<instance part="IC1" gate="PORTA_L" x="116.84" y="111.76" rot="MR0"/>
+<instance part="IC1" gate="PORTA_L" x="119.38" y="111.76" rot="MR0"/>
 <instance part="IC1" gate="AN_POWER" x="58.42" y="20.32"/>
 <instance part="IC1" gate="G$2" x="43.18" y="20.32"/>
@@
 <segment>
 <pinref part="IC1" gate="PORTA_L" pin="PA7"/>
-<wire x1="124.46" y1="101.6" x2="129.54" y2="101.6" width="0.1524" layer="91"/>
-<label x="129.54" y="101.6" size="1.27" layer="95" xref="yes"/>
+<wire x1="127" y1="101.6" x2="132.08" y2="101.6" width="0.1524" layer="91"/>
+<label x="132.08" y="101.6" size="1.27" layer="95" xref="yes"/>
 </segment>
 </net>
@@
 <segment>
 <pinref part="IC1" gate="PORTA_L" pin="PA6"/>
-<wire x1="124.46" y1="104.14" x2="129.54" y2="104.14" width="0.1524" layer="91"/>
-<label x="129.54" y="104.14" size="1.27" layer="95" xref="yes"/>
+<wire x1="127" y1="104.14" x2="132.08" y2="104.14" width="0.1524" layer="91"/>
+<label x="132.08" y="104.14" size="1.27" layer="95" xref="yes"/>
 </segment>
 </net>
@@
 <segment>
 <pinref part="IC1" gate="PORTA_L" pin="PA5"/>
-<wire x1="124.46" y1="106.68" x2="129.54" y2="106.68" width="0.1524" layer="91"/>
-<label x="129.54" y="106.68" size="1.27" layer="95" xref="yes"/>
+<wire x1="127" y1="106.68" x2="132.08" y2="106.68" width="0.1524" layer="91"/>
+<label x="132.08" y="106.68" size="1.27" layer="95" xref="yes"/>
 </segment>
 </net>
@@
 <label x="88.9" y="154.94" size="0.762" layer="95" rot="R270" xref="yes"/>
 </segment>
+<segment>
+<pinref part="IC1" gate="PORTA_L" pin="PA0"/>
+<wire x1="127" y1="119.38" x2="129.54" y2="119.38" width="0.1524" layer="91"/>
+<label x="129.54" y="119.38" size="1.27" layer="95" xref="yes"/>
+</segment>
 </net>
 <net name="N$23" class="0">
@@
 <junction x="45.72" y="154.94"/>
 </segment>
+<segment>
+<pinref part="IC1" gate="PORTB_L" pin="PB6"/>
+<wire x1="93.98" y1="106.68" x2="96.52" y2="106.68" width="0.1524" layer="91"/>
+<label x="96.52" y="106.68" size="1.27" layer="95" xref="yes"/>
+</segment>
 </net>
 <net name="N$1" class="0">
@@
 <segment>
 <pinref part="IC1" gate="PORTA_L" pin="PA2"/>
-<wire x1="124.46" y1="114.3" x2="127" y2="114.3" width="0.1524" layer="91"/>
-<label x="127" y="114.3" size="1.27" layer="95" xref="yes"/>
+<wire x1="127" y1="114.3" x2="129.54" y2="114.3" width="0.1524" layer="91"/>
+<label x="129.54" y="114.3" size="1.27" layer="95" xref="yes"/>
 </segment>
 </net>
@@
 <segment>
 <pinref part="IC1" gate="PORTA_L" pin="PA3"/>
-<wire x1="124.46" y1="111.76" x2="127" y2="111.76" width="0.1524" layer="91"/>
-<label x="127" y="111.76" size="1.27" layer="95" xref="yes"/>
-</segment>
-</net>
+<wire x1="127" y1="111.76" x2="129.54" y2="111.76" width="0.1524" layer="91"/>
+<label x="129.54" y="111.76" size="1.27" layer="95" xref="yes"/>
+</segment>
+</net>
